File: mouse_joystick_controller/mouse_joystick_controller.kicad_pcb (KiCad board)
At the start: 4 copper layers, 38 parts, among them J1 Conn_TERM_HDR_01x02_Pin_3.5MM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, J2 5.5x2.5_SMD_RA, J3 5.5x2.1_SMD_RA, J4 Conn_FFC_20_Pin_1mm_bottom-ZF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, U1 TMC429, U2 NCR421ZX, U3 3.3V_150MA, U4 AD9837ACPZ-RL, U5 PGA305ARHHR, U6 LVDS_4-4_HALF_DS91M040TSQE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

Commit message: Move standby pin
Connections:
- J4 pad 10: /motors/driver_0/REF_B -> /motors/driver_0/STANDBY_B
- J4 pad 5: /motors/driver_0/STANDBY_A -> /motors/driver_0/REFR_A
- J4 pad 6: /motors/driver_0/STANDBY_B -> /motors/driver_0/REFR_B
- J4 pad 7: /motors/driver_0/REFR_A -> /motors/driver_0/REF_A
- J4 pad 8: /motors/driver_0/REFR_B -> /motors/driver_0/REF_B
- J4 pad 9: /motors/driver_0/REF_A -> /motors/driver_0/STANDBY_A
- R7 pad 1: /motors/driver_0/REF_A -> /motors/driver_0/STANDBY_A
- R7 pad 2: /motors/driver_0/REF_B -> /motors/driver_0/STANDBY_B
- R8 pad 1: /motors/driver_0/REFR_A -> /motors/driver_0/REF_A
- R8 pad 2: /motors/driver_0/REFR_B -> /motors/driver_0/REF_B
- R9 pad 1: /motors/driver_0/STANDBY_A -> /motors/driver_0/REFR_A
- R9 pad 2: /motors/driver_0/STANDBY_B -> /motors/driver_0/REFR_B
- U7 pad 15: unconnected-(U7-~{RE3}-Pad15) -> /motors/GND
- U7 pad 16: /motors/+3.3V -> unconnected-(U7-DE3-Pad16)
- U7 pad 17: /motors/driver_0/STANDBY_A -> /motors/driver_0/REFR_A
- U7 pad 18: /motors/driver_0/STANDBY_B -> /motors/driver_0/REFR_B
- U7 pad 19: /motors/driver_0/REFR_A -> /motors/driver_0/REF_A
- U7 pad 20: /motors/driver_0/REFR_B -> /motors/driver_0/REF_B
- U7 pad 21: /motors/driver_0/REF_A -> /motors/driver_0/STANDBY_A
- U7 pad 22: /motors/driver_0/REF_B -> /motors/driver_0/STANDBY_B
- U7 pad 27: unconnected-(U7-DE1-Pad27) -> /motors/+3.3V
- U7 pad 28: /motors/GND -> unconnected-(U7-~{RE1}-Pad28)
- U7 pad 3: /motors/REF_0 -> unconnected-(U7-RO1-Pad3)
- U7 pad 4: /motors/GND -> /motors/STANDBY_0
- U7 pad 5: /motors/REFR_0 -> /motors/REF_0
- U7 pad 7: unconnected-(U7-RO3-Pad7) -> /motors/REFR_0
- U7 pad 8: /motors/STANDBY_0 -> /motors/GND
Changed lines of the file:
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@@
   (title_block
     (title "mouse_joystick_controller")
-    (date "2023-05-24")
+    (date "2023-07-12")
     (rev "2.0")
     (company "Howard Hughes Medical Institute")
@@
   (net 113 "unconnected-(U6-FSEN1-Pad32)")
   (net 114 "unconnected-(U7-RO0-Pad1)")
-  (net 115 "unconnected-(U7-RO3-Pad7)")
+  (net 115 "unconnected-(U7-RO1-Pad3)")
   (net 116 "/motors/STANDBY_0")
   (net 117 "unconnected-(U7-FSEN2-Pad9)")
   (net 118 "unconnected-(U7-DE2-Pad14)")
-  (net 119 "unconnected-(U7-~{RE3}-Pad15)")
+  (net 119 "unconnected-(U7-DE3-Pad16)")
   (net 120 "unconnected-(U7-~{RE0}-Pad26)")
-  (net 121 "unconnected-(U7-DE1-Pad27)")
+  (net 121 "unconnected-(U7-~{RE1}-Pad28)")
   (net 122 "unconnected-(U7-FSEN1-Pad32)")
   (net 123 "/microcontroller/GND")
@@
       (net 69 "/motors/+24V") (pinfunction "Pin_4") (pintype "passive"))
     (pad "5" smd rect (at -5.5 0) (size 0.6 1.8) (layers "F.Cu" "F.Paste" "F.Mask")
-      (net 70 "/motors/driver_0/STANDBY_A") (pinfunction "Pin_5") (pintype "passive"))
+      (net 8 "/motors/driver_0/REFR_A") (pinfunction "Pin_5") (pintype "passive"))
     (pad "6" smd rect (at -4.5 0) (size 0.6 1.8) (layers "F.Cu" "F.Paste" "F.Mask")
-      (net 71 "/motors/driver_0/STANDBY_B") (pinfunction "Pin_6") (pintype "passive"))
+      (net 9 "/motors/driver_0/REFR_B") (pinfunction "Pin_6") (pintype "passive"))
     (pad "7" smd rect (at -3.5 0) (size 0.6 1.8) (layers "F.Cu" "F.Paste" "F.Mask")
-      (net 8 "/motors/driver_0/REFR_A") (pinfunction "Pin_7") (pintype "passive"))
+      (net 10 "/motors/driver_0/REF_A") (pinfunction "Pin_7") (pintype "passive"))
     (pad "8" smd rect (at -2.5 0) (size 0.6 1.8) (layers "F.Cu" "F.Paste" "F.Mask")
-      (net 9 "/motors/driver_0/REFR_B") (pinfunction "Pin_8") (pintype "passive"))
+      (net 11 "/motors/driver_0/REF_B") (pinfunction "Pin_8") (pintype "passive"))
     (pad "9" smd rect (at -1.5 0) (size 0.6 1.8) (layers "F.Cu" "F.Paste" "F.Mask")
-      (net 10 "/motors/driver_0/REF_A") (pinfunction "Pin_9") (pintype "passive"))
+      (net 70 "/motors/driver_0/STANDBY_A") (pinfunction "Pin_9") (pintype "passive"))
     (pad "10" smd rect (at -0.5 0) (size 0.6 1.8) (layers "F.Cu" "F.Paste" "F.Mask")
-      (net 11 "/motors/driver_0/REF_B") (pinfunction "Pin_10") (pintype "passive"))
+      (net 71 "/motors/driver_0/STANDBY_B") (pinfunction "Pin_10") (pintype "passive"))
     (pad "11" smd rect (at 0.5 0) (size 0.6 1.8) (layers "F.Cu" "F.Paste" "F.Mask")
       (net 12 "/motors/driver_0/~{DRIVER_ENABLE_A}") (pinfunction "Pin_11") (pintype "passive"))
@@
       (stroke (width 0.1) (type solid)) (layer "F.Fab"))
     (pad "1" smd roundrect (at -0.51 0) (size 0.54 0.64) (layers "F.Cu" "F.Paste" "F.Mask") (roundrect_rratio 0.25)
-      (net 70 "/motors/driver_0/STANDBY_A") (pintype "passive"))
+      (net 8 "/motors/driver_0/REFR_A") (pintype "passive"))
     (pad "2" smd roundrect (at 0.51 0) (size 0.54 0.64) (layers "F.Cu" "F.Paste" "F.Mask") (roundrect_rratio 0.25)
-      (net 71 "/motors/driver_0/STANDBY_B") (pintype "passive"))
+      (net 9 "/motors/driver_0/REFR_B") (pintype "passive"))
     (model "${KICAD_USER_DIR}/packages3D/Janelia.3dshapes/R_0402_1005Metric.step"
       (offset (xyz 0 0 0))
@@
       (stroke (width 0.1) (type solid)) (layer "F.Fab"))
     (pad "1" smd roundrect (at -0.51 0) (size 0.54 0.64) (layers "F.Cu" "F.Paste" "F.Mask") (roundrect_rratio 0.25)
-      (net 10 "/motors/driver_0/REF_A") (pintype "passive"))
+      (net 70 "/motors/driver_0/STANDBY_A") (pintype "passive"))
     (pad "2" smd roundrect (at 0.51 0) (size 0.54 0.64) (layers "F.Cu" "F.Paste" "F.Mask") (roundrect_rratio 0.25)
-      (net 11 "/motors/driver_0/REF_B") (pintype "passive"))
+      (net 71 "/motors/driver_0/STANDBY_B") (pintype "passive"))
     (model "${KICAD_USER_DIR}/packages3D/Janelia.3dshapes/R_0402_1005Metric.step"
       (offset (xyz 0 0 0))
@@
       (net 60 "/motors/~{DRIVER_ENABLE_0}") (pinfunction "DI0") (pintype "input"))
     (pad "3" smd roundrect (at -2.4 -0.75 90) (size 0.24 0.6) (layers "F.Cu" "F.Paste" "F.Mask") (roundrect_rratio 0.1)
-      (net 61 "/motors/REF_0") (pinfunction "RO1") (pintype "output"))
+      (net 115 "unconnected-(U7-RO1-Pad3)") (pinfunction "RO1") (pintype "output+no_connect"))
     (pad "4" smd roundrect (at -2.4 -0.25 90) (size 0.24 0.6) (layers "F.Cu" "F.Paste" "F.Mask") (roundrect_rratio 0.1)
-      (net 5 "/motors/GND") (pinfunction "DI1") (pintype "input"))
+      (net 116 "/motors/STANDBY_0") (pinfunction "DI1") (pintype "input"))
     (pad "5" smd roundrect (at -2.4 0.25 90) (size 0.24 0.6) (layers "F.Cu" "F.Paste" "F.Mask") (roundrect_rratio 0.1)
-      (net 62 "/motors/REFR_0") (pinfunction "RO2") (pintype "output"))
+      (net 61 "/motors/REF_0") (pinfunction "RO2") (pintype "output"))
     (pad "6" smd roundrect (at -2.4 0.75 90) (size 0.24 0.6) (layers "F.Cu" "F.Paste" "F.Mask") (roundrect_rratio 0.1)
       (net 5 "/motors/GND") (pinfunction "DI2") (pintype "input"))
     (pad "7" smd roundrect (at -2.4 1.25 90) (size 0.24 0.6) (layers "F.Cu" "F.Paste" "F.Mask") (roundrect_rratio 0.1)
-      (net 115 "unconnected-(U7-RO3-Pad7)") (pinfunction "RO3") (pintype "output+no_connect"))
+      (net 62 "/motors/REFR_0") (pinfunction "RO3") (pintype "output"))
     (pad "8" smd roundrect (at -2.4 1.75 90) (size 0.24 0.6) (layers "F.Cu" "F.Paste" "F.Mask") (roundrect_rratio 0.1)
-      (net 116 "/motors/STANDBY_0") (pinfunction "DI3") (pintype "input"))
+      (net 5 "/motors/GND") (pinfunction "DI3") (pintype "input"))
     (pad "9" smd roundrect (at -1.75 2.4) (size 0.24 0.6) (layers "F.Cu" "F.Paste" "F.Mask") (roundrect_rratio 0.1)
       (net 117 "unconnected-(U7-FSEN2-Pad9)") (pinfunction "FSEN2") (pintype "input+no_connect"))
@@
       (net 118 "unconnected-(U7-DE2-Pad14)") (pinfunction "DE2") (pintype "input+no_connect"))
     (pad "15" smd roundrect (at 1.25 2.4) (size 0.24 0.6) (layers "F.Cu" "F.Paste" "F.Mask") (roundrect_rratio 0.1)
-      (net 119 "unconnected-(U7-~{RE3}-Pad15)") (pinfunction "~{RE3}") (pintype "input+no_connect"))
+      (net 5 "/motors/GND") (pinfunction "~{RE3}") (pintype "input"))
     (pad "16" smd roundrect (at 1.75 2.4) (size 0.24 0.6) (layers "F.Cu" "F.Paste" "F.Mask") (roundrect_rratio 0.1)
-      (net 4 "/motors/+3.3V") (pinfunction "DE3") (pintype "input"))
+      (net 119 "unconnected-(U7-DE3-Pad16)") (pinfunction "DE3") (pintype "input+no_connect"))
     (pad "17" smd roundrect (at 2.4 1.75 90) (size 0.24 0.6) (layers "F.Cu" "F.Paste" "F.Mask") (roundrect_rratio 0.1)
-      (net 70 "/motors/driver_0/STANDBY_A") (pinfunction "A3") (pintype "bidirectional"))
+      (net 8 "/motors/driver_0/REFR_A") (pinfunction "A3") (pintype "bidirectional"))
     (pad "18" smd roundrect (at 2.4 1.25 90) (size 0.24 0.6) (layers "F.Cu" "F.Paste" "F.Mask") (roundrect_rratio 0.1)
-      (net 71 "/motors/driver_0/STANDBY_B") (pinfunction "B3") (pintype "bidirectional"))
+      (net 9 "/motors/driver_0/REFR_B") (pinfunction "B3") (pintype "bidirectional"))
     (pad "19" smd roundrect (at 2.4 0.75 90) (size 0.24 0.6) (layers "F.Cu" "F.Paste" "F.Mask") (roundrect_rratio 0.1)
-      (net 8 "/motors/driver_0/REFR_A") (pinfunction "A2") (pintype "bidirectional"))
+      (net 10 "/motors/driver_0/REF_A") (pinfunction "A2") (pintype "bidirectional"))
     (pad "20" smd roundrect (at 2.4 0.25 90) (size 0.24 0.6) (layers "F.Cu" "F.Paste" "F.Mask") (roundrect_rratio 0.1)
-      (net 9 "/motors/driver_0/REFR_B") (pinfunction "B2") (pintype "bidirectional"))
+      (net 11 "/motors/driver_0/REF_B") (pinfunction "B2") (pintype "bidirectional"))
     (pad "21" smd roundrect (at 2.4 -0.25 90) (size 0.24 0.6) (layers "F.Cu" "F.Paste" "F.Mask") (roundrect_rratio 0.1)
-      (net 10 "/motors/driver_0/REF_A") (pinfunction "A1") (pintype "bidirectional"))
+      (net 70 "/motors/driver_0/STANDBY_A") (pinfunction "A1") (pintype "bidirectional"))
     (pad "22" smd roundrect (at 2.4 -0.75 90) (size 0.24 0.6) (layers "F.Cu" "F.Paste" "F.Mask") (roundrect_rratio 0.1)
-      (net 11 "/motors/driver_0/REF_B") (pinfunction "B1") (pintype "bidirectional"))
+      (net 71 "/motors/driver_0/STANDBY_B") (pinfunction "B1") (pintype "bidirectional"))
     (pad "23" smd roundrect (at 2.4 -1.25 90) (size 0.24 0.6) (layers "F.Cu" "F.Paste" "F.Mask") (roundrect_rratio 0.1)
       (net 12 "/motors/driver_0/~{DRIVER_ENABLE_A}") (pinfunction "A0") (pintype "bidirectional"))
@@
       (net 120 "unconnected-(U7-~{RE0}-Pad26)") (pinfunction "~{RE0}") (pintype "input+no_connect"))
     (pad "27" smd roundrect (at 0.75 -2.4) (size 0.24 0.6) (layers "F.Cu" "F.Paste" "F.Mask") (roundrect_rratio 0.1)
-      (net 121 "unconnected-(U7-DE1-Pad27)") (pinfunction "DE1") (pintype "input+no_connect"))
+      (net 4 "/motors/+3.3V") (pinfunction "DE1") (pintype "input"))
     (pad "28" smd roundrect (at 0.25 -2.4) (size 0.24 0.6) (layers "F.Cu" "F.Paste" "F.Mask") (roundrect_rratio 0.1)
-      (net 5 "/motors/GND") (pinfunction "~{RE1}") (pintype "input"))
+      (net 121 "unconnected-(U7-~{RE1}-Pad28)") (pinfunction "~{RE1}") (pintype "input+no_connect"))
     (pad "29" smd roundrect (at -0.25 -2.4) (size 0.24 0.6) (layers "F.Cu" "F.Paste" "F.Mask") (roundrect_rratio 0.1)
       (net 4 "/motors/+3.3V") (pinfunction "VDD") (pintype "power_in"))
@@
       (stroke (width 0.1) (type solid)) (layer "F.Fab"))
     (pad "1" smd roundrect (at -0.51 0) (size 0.54 0.64) (layers "F.Cu" "F.Paste" "F.Mask") (roundrect_rratio 0.25)
-      (net 8 "/motors/driver_0/REFR_A") (pintype "passive"))
+      (net 10 "/motors/driver_0/REF_A") (pintype "passive"))
     (pad "2" smd roundrect (at 0.51 0) (size 0.54 0.64) (layers "F.Cu" "F.Paste" "F.Mask") (roundrect_rratio 0.25)
-      (net 9 "/motors/driver_0/REFR_B") (pintype "passive"))
+      (net 11 "/motors/driver_0/REF_B") (pintype "passive"))
     (model "${KICAD_USER_DIR}/packages3D/Janelia.3dshapes/R_0402_1005Metric.step"
       (offset (xyz 0 0 0))
