File: mouse_joystick_controller/lickport.kicad_sch (KiCad schematic)
At the start: 0 parts

Commit message: Rearrange sheets
Other:
- company: (none) -> Howard Hughes Medical Institute
- title: (none) -> mouse_joystick_controller
Changed lines of the file:
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@@
 (kicad_sch (version 20230121) (generator eeschema)
   (paper "A4")
+  (title_block
+    (title "mouse_joystick_controller")
+    (date "2023-05-24")
+    (rev "2.0")
+    (company "Howard Hughes Medical Institute")
+  )
 )
