File: mouse_joystick_controller/microcontroller.kicad_sch (KiCad schematic)
At the start: 1 part

Commit message: Change brake circuitry again
Other:
- company: (none) -> Howard Hughes Medical Institute
- title: (none) -> mouse_joystick_controller
Changed lines of the file:
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@@
 (kicad_sch (version 20230121) (generator eeschema)
   (paper "A4")
+  (title_block
+    (title "mouse_joystick_controller")
+    (date "2023-06-02")
+    (rev "2.0")
+    (company "Howard Hughes Medical Institute")
+  )
   (symbol (lib_id "Janelia:TEENSY_4.1_HEADERS") (at 134.62 78.74 0) (unit 1)
     (in_bom yes) (on_board yes) (dnp no) (fields_autoplaced)

Commit message: Remove teensy component
Parts:
- removed TEENSY1: TEENSY_4.1_HEADERS, Janelia:TEENSY_4.1_HEADERS, symbol Janelia:TEENSY_4.1_HEADERS
Changed lines of the file:
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@@
     (company "Howard Hughes Medical Institute")
   )
-  (symbol (lib_id "Janelia:TEENSY_4.1_HEADERS") (at 134.62 78.74 0) (unit 1)
-    (in_bom yes) (on_board yes) (dnp no) (fields_autoplaced)
-    (property "Reference" "TEENSY1" (at 134.62 57.15 0)
-      (effects (font (size 1.524 1.524)))
-    )
-    (property "Value" "TEENSY_4.1_HEADERS" (at 134.62 59.69 0)
-      (effects (font (size 1.524 1.524)))
-    )
-    (property "Footprint" "Janelia:TEENSY_4.1_HEADERS" (at 134.62 52.07 0)
-      (effects (font (size 1.524 1.524)) hide)
-    )
-    (property "Datasheet" "" (at 135.89 8.89 0)
-      (effects (font (size 1.524 1.524)))
-    )
-    (property "Vendor" "Digi-Key" (at 134.62 49.53 0)
-      (effects (font (size 1.524 1.524)) hide)
-    )
-    (property "Vendor Part Number" "S7057-ND" (at 134.62 46.99 0)
-      (effects (font (size 1.524 1.524)) hide)
-    )
-    (property "Description" "CONN HDR 24POS 0.1 GOLD PCB" (at 134.62 44.45 0)
-      (effects (font (size 1.524 1.524)) hide)
-    )
-    (property "Manufacturer" "Sullins Connector Solutions" (at 134.62 78.74 0)
-      (effects (font (size 1.27 1.27)) hide)
-    )
-    (property "Manufacturer Part Number" "PPPC241LFBN-RC" (at 134.62 78.74 0)
-      (effects (font (size 1.27 1.27)) hide)
-    )
-    (pin "0")
-    (pin "1")
-    (pin "10")
-    (pin "11")
-    (pin "12")
-    (pin "13")
-    (pin "14")
-    (pin "15")
-    (pin "16")
-    (pin "17")
-    (pin "18")
-    (pin "19")
-    (pin "2")
-    (pin "20")
-    (pin "21")
-    (pin "22")
-    (pin "23")
-    (pin "24")
-    (pin "25")
-    (pin "26")
-    (pin "27")
-    (pin "28")
-    (pin "29")
-    (pin "3")
-    (pin "30")
-    (pin "31")
-    (pin "32")
-    (pin "33")
-    (pin "34")
-    (pin "35")
-    (pin "36")
-    (pin "37")
-    (pin "38")
-    (pin "39")
-    (pin "3V3")
-    (pin "4")
-    (pin "40")
-    (pin "41")
-    (pin "5")
-    (pin "6")
-    (pin "7")
-    (pin "8")
-    (pin "9")
-    (pin "GND")
-    (pin "V")
-    (instances
-      (project "mouse_joystick_controller"
-        (path "/cc457ebc-4af6-4663-b19f-8cb38f061cb4/6a52ceec-773f-4608-99f1-9264727759c9"
-          (reference "TEENSY1") (unit 1)
-        )
-      )
-    )
-  )
 )

Commit message: Test pin rcpt
Parts:
- added A1: TEENSY_4.1_PIN_RECEPTACLES, Janelia:TEENSY_4.1_PIN_RECEPTACLES, symbol Janelia:TEENSY_4.1_PIN_RECEPTACLES
- added PR0, PR1: Conn_Pin_Rcpt-0305-1-15, Janelia:CONN_PIN_RCPT-0305-1-15, symbol Janelia:Conn_Pin_Rcpt-0305-1-15
Connections:
- new net D0: PR1.1 (Pin_1)
- new net GND: PR0.1 (Pin_1)
Changed lines of the file:
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@@
   (title_block
     (title "mouse_joystick_controller")
-    (date "2023-06-07")
+    (date "2023-06-09")
     (rev "2.0")
     (company "Howard Hughes Medical Institute")
   )
+  (wire (pts (xy 102.87 66.04) (xy 105.41 66.04))
+    (stroke (width 0) (type default))
+  )
+  (wire (pts (xy 102.87 68.58) (xy 105.41 68.58))
+    (stroke (width 0) (type default))
+  )
+  (label "GND" (at 102.87 66.04 180) (fields_autoplaced)
+    (effects (font (size 1.27 1.27)) (justify right bottom))
+  )
+  (label "D0" (at 102.87 68.58 180) (fields_autoplaced)
+    (effects (font (size 1.27 1.27)) (justify right bottom))
+  )
+  (symbol (lib_id "Janelia:Conn_Pin_Rcpt-0305-1-15") (at 111.76 66.04 0) (unit 1)
+    (in_bom yes) (on_board yes) (dnp no)
+    (property "Reference" "PR0" (at 107.95 64.77 0) (do_not_autoplace)
+      (effects (font (size 1.27 1.27)))
+    )
+    (property "Value" "Conn_Pin_Rcpt-0305-1-15" (at 111.76 45.72 0) (do_not_autoplace)
+      (effects (font (size 1.27 1.27)) hide)
+    )
+    (property "Footprint" "Janelia:CONN_PIN_RCPT-0305-1-15" (at 111.76 60.96 0)
+      (effects (font (size 1.27 1.27)) hide)
+    )
+    (property "Datasheet" "~" (at 111.76 57.15 0) (do_not_autoplace)
+      (effects (font (size 1.27 1.27)) hide)
+    )
+    (property "Description" "CONN PIN RCPT .025-.037 SOLDER" (at 111.76 53.34 0)
+      (effects (font (size 1.27 1.27)) hide)
+    )
+    (property "Manufacturer" "Mill-Max Manufacturing Corp." (at 111.76 50.8 0)
+      (effects (font (size 1.27 1.27)) hide)
+    )
+    (property "Manufacturer Part Number" "0305-1-15-15-47-27-10-0" (at 111.76 55.88 0)
+      (effects (font (size 1.27 1.27)) hide)
+    )
+    (property "Vendor" "Digi-Key" (at 111.76 48.26 0)
+      (effects (font (size 1.27 1.27)) hide)
+    )
+    (property "Vendor Part Number" "ED90332-ND" (at 111.76 58.42 0)
+      (effects (font (size 1.27 1.27)) hide)
+    )
+    (pin "1")
+    (instances
+      (project "mouse_joystick_controller"
+        (path "/cc457ebc-4af6-4663-b19f-8cb38f061cb4/6a52ceec-773f-4608-99f1-9264727759c9"
+          (reference "PR0") (unit 1)
+        )
+      )
+    )
+  )
+  (symbol (lib_id "Janelia:TEENSY_4.1_PIN_RECEPTACLES") (at 138.43 82.55 0) (unit 1)
+    (in_bom no) (on_board yes) (dnp no) (fields_autoplaced)
+    (property "Reference" "A1" (at 138.43 63.5 0) (do_not_autoplace)
+      (effects (font (size 1.524 1.524)))
+    )
+    (property "Value" "TEENSY_4.1_PIN_RECEPTACLES" (at 138.43 52.07 0)
+      (effects (font (size 1.524 1.524)) hide)
+    )
+    (property "Footprint" "Janelia:TEENSY_4.1_PIN_RECEPTACLES" (at 138.43 55.88 0)
+      (effects (font (size 1.524 1.524)) hide)
+    )
+    (property "Datasheet" "" (at 139.7 12.7 0)
+      (effects (font (size 1.524 1.524)))
+    )
+    (property "Sim.Enable" "0" (at 138.43 82.55 0)
+      (effects (font (size 1.27 1.27)) hide)
+    )
+    (instances
+      (project "mouse_joystick_controller"
+        (path "/cc457ebc-4af6-4663-b19f-8cb38f061cb4/6a52ceec-773f-4608-99f1-9264727759c9"
+          (reference "A1") (unit 1)
+        )
+      )
+    )
+  )
+  (symbol (lib_id "Janelia:Conn_Pin_Rcpt-0305-1-15") (at 111.76 68.58 0) (unit 1)
+    (in_bom yes) (on_board yes) (dnp no)
+    (property "Reference" "PR1" (at 107.95 67.31 0) (do_not_autoplace)
+      (effects (font (size 1.27 1.27)))
+    )
+    (property "Value" "Conn_Pin_Rcpt-0305-1-15" (at 111.76 48.26 0) (do_not_autoplace)
+      (effects (font (size 1.27 1.27)) hide)
+    )
+    (property "Footprint" "Janelia:CONN_PIN_RCPT-0305-1-15" (at 111.76 63.5 0)
+      (effects (font (size 1.27 1.27)) hide)
+    )
+    (property "Datasheet" "~" (at 111.76 59.69 0) (do_not_autoplace)
+      (effects (font (size 1.27 1.27)) hide)
+    )
+    (property "Description" "CONN PIN RCPT .025-.037 SOLDER" (at 111.76 55.88 0)
+      (effects (font (size 1.27 1.27)) hide)
+    )
+    (property "Manufacturer" "Mill-Max Manufacturing Corp." (at 111.76 53.34 0)
+      (effects (font (size 1.27 1.27)) hide)
+    )
+    (property "Manufacturer Part Number" "0305-1-15-15-47-27-10-0" (at 111.76 58.42 0)
+      (effects (font (size 1.27 1.27)) hide)
+    )
+    (property "Vendor" "Digi-Key" (at 111.76 50.8 0)
+      (effects (font (size 1.27 1.27)) hide)
+    )
+    (property "Vendor Part Number" "ED90332-ND" (at 111.76 60.96 0)
+      (effects (font (size 1.27 1.27)) hide)
+    )
+    (pin "1")
+    (instances
+      (project "mouse_joystick_controller"
+        (path "/cc457ebc-4af6-4663-b19f-8cb38f061cb4/6a52ceec-773f-4608-99f1-9264727759c9"
+          (reference "PR1") (unit 1)
+        )
+      )
+    )
+  )
 )
