File: mouse_joystick_controller/power.kicad_sch (KiCad schematic)
At the start: 5 parts, among them J3 5.5x2.5_SMD_RA, J4 5.5x2.1_SMD_RA, U6 3.3V_150MA

Commit message: Test pin rcpt
Parts:
- renumbered J3 to J2, J4 to J3, U6 to U3
Changed lines of the file:
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@@
   (title_block
     (title "mouse_joystick_controller")
-    (date "2023-06-07")
+    (date "2023-06-09")
     (rev "2.0")
     (company "Howard Hughes Medical Institute")
@@
         )
         (path "/cc457ebc-4af6-4663-b19f-8cb38f061cb4/f62b8726-10b6-4dce-a8d7-bdccf22557c3"
-          (reference "C2") (unit 1)
+          (reference "C4") (unit 1)
         )
       )
@@
   (symbol (lib_id "Janelia:Barrel_Jack_Switch_5.5x2.5_SMD_RA_54-00165") (at 154.94 59.69 0) (unit 1)
     (in_bom yes) (on_board yes) (dnp no)
-    (property "Reference" "J3" (at 154.94 54.61 0)
+    (property "Reference" "J2" (at 154.94 54.61 0)
       (effects (font (size 1.27 1.27)))
     )
@@
       (effects (font (size 1.27 1.27)) hide)
     )
+    (property "Sim.Enable" "0" (at 154.94 59.69 0)
+      (effects (font (size 1.27 1.27)) hide)
+    )
     (pin "1")
     (pin "2")
@@
       (project "mouse_joystick_controller"
         (path "/cc457ebc-4af6-4663-b19f-8cb38f061cb4/f62b8726-10b6-4dce-a8d7-bdccf22557c3"
-          (reference "J3") (unit 1)
+          (reference "J2") (unit 1)
         )
       )
@@
         )
         (path "/cc457ebc-4af6-4663-b19f-8cb38f061cb4/f62b8726-10b6-4dce-a8d7-bdccf22557c3"
-          (reference "C1") (unit 1)
+          (reference "C3") (unit 1)
         )
       )
@@
   (symbol (lib_id "Janelia:Regulator_Linear_3.3V_150MA_30Vin") (at 163.83 93.98 0) (unit 1)
     (in_bom yes) (on_board yes) (dnp no)
-    (property "Reference" "U6" (at 170.18 101.6 0)
+    (property "Reference" "U3" (at 170.18 101.6 0)
       (effects (font (size 1.524 1.524)))
     )
@@
     )
     (property "Description" "IC REG LINEAR 3.3V 150MA" (at 163.83 76.2 0)
+      (effects (font (size 1.27 1.27)) hide)
+    )
+    (property "Sim.Enable" "0" (at 163.83 93.98 0)
       (effects (font (size 1.27 1.27)) hide)
     )
@@
       (project "mouse_joystick_controller"
         (path "/cc457ebc-4af6-4663-b19f-8cb38f061cb4/f62b8726-10b6-4dce-a8d7-bdccf22557c3"
-          (reference "U6") (unit 1)
+          (reference "U3") (unit 1)
         )
       )
@@
   (symbol (lib_id "Janelia:Barrel_Jack_Switch_5.5x2.1_SMD_RA_54-00164") (at 184.15 59.69 0) (unit 1)
     (in_bom yes) (on_board yes) (dnp no)
-    (property "Reference" "J4" (at 184.15 54.61 0)
+    (property "Reference" "J3" (at 184.15 54.61 0)
       (effects (font (size 1.27 1.27)))
     )
@@
       (effects (font (size 1.27 1.27)) hide)
     )
+    (property "Sim.Enable" "0" (at 184.15 59.69 0)
+      (effects (font (size 1.27 1.27)) hide)
+    )
     (pin "1")
     (pin "2")
@@
       (project "mouse_joystick_controller"
         (path "/cc457ebc-4af6-4663-b19f-8cb38f061cb4/f62b8726-10b6-4dce-a8d7-bdccf22557c3"
-          (reference "J4") (unit 1)
-        )
-      )
+          (reference "J3") (unit 1)
+        )
+      )

Commit message: Update to kicad 7.0.8
Parts:
- removed J2: 5.5x2.5_SMD_RA, Janelia:CONN_54-00165, symbol Janelia:Barrel_Jack_Switch_5.5x2.5_SMD_RA_54-00165
Connections:
- net +30V is gone; now on net +24V: J3.1
- no-connect marks 3 -> 2
Changed lines of the file:
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@@
   (title_block
     (title "mouse_joystick_controller")
-    (date "2023-07-12")
+    (date "2023-10-13")
     (rev "2.0")
     (company "Howard Hughes Medical Institute")
   )
-  (no_connect (at 162.56 59.69))
   (no_connect (at 151.13 99.06))
   (no_connect (at 191.77 59.69))
@@
     (stroke (width 0) (type default))
   )
-  (wire (pts (xy 165.1 62.23) (xy 162.56 62.23))
-    (stroke (width 0) (type default))
-  )
   (wire (pts (xy 135.89 101.6) (xy 135.89 104.14))
     (stroke (width 0) (type default))
   )
   (wire (pts (xy 135.89 88.9) (xy 135.89 91.44))
-    (stroke (width 0) (type default))
-  )
-  (wire (pts (xy 83.82 88.9) (xy 81.28 88.9))
     (stroke (width 0) (type default))
   )
@@
     (stroke (width 0) (type default))
   )
-  (wire (pts (xy 165.1 57.15) (xy 162.56 57.15))
-    (stroke (width 0) (type default))
-  )
   (wire (pts (xy 148.59 93.98) (xy 151.13 93.98))
     (stroke (width 0) (type default))
@@
   (label "GND" (at 165.1 107.95 270) (fields_autoplaced)
     (effects (font (size 1.27 1.27)) (justify right bottom))
-  )
-  (label "+30V" (at 83.82 88.9 0) (fields_autoplaced)
-    (effects (font (size 1.27 1.27)) (justify left bottom))
   )
   (label "+24V" (at 148.59 93.98 180) (fields_autoplaced)
@@
     (effects (font (size 1.27 1.27)) (justify left bottom))
   )
-  (label "+24V" (at 165.1 57.15 0) (fields_autoplaced)
-    (effects (font (size 1.27 1.27)) (justify left bottom))
-  )
-  (label "GND" (at 165.1 62.23 0) (fields_autoplaced)
+  (label "+24V" (at 194.31 57.15 0) (fields_autoplaced)
     (effects (font (size 1.27 1.27)) (justify left bottom))
   )
@@
     (effects (font (size 1.27 1.27)) (justify left bottom))
   )
-  (label "+30V" (at 194.31 57.15 0) (fields_autoplaced)
-    (effects (font (size 1.27 1.27)) (justify left bottom))
-  )
   (hierarchical_label "GND" (shape passive) (at 81.28 100.33 180) (fields_autoplaced)
-    (effects (font (size 1.27 1.27)) (justify right))
-  )
-  (hierarchical_label "+30V" (shape passive) (at 81.28 88.9 180) (fields_autoplaced)
     (effects (font (size 1.27 1.27)) (justify right))
   )
@@
         )
       )
-    )
-  )
-  (symbol (lib_id "Janelia:Barrel_Jack_Switch_5.5x2.5_SMD_RA_54-00165") (at 154.94 59.69 0) (unit 1)
-    (in_bom yes) (on_board yes) (dnp no)
-    (property "Reference" "J2" (at 154.94 54.61 0)
-      (effects (font (size 1.27 1.27)))
-    )
-    (property "Value" "5.5x2.5_SMD_RA" (at 154.94 64.77 0)
-      (effects (font (size 1.27 1.27)))
-    )
-    (property "Footprint" "Janelia:CONN_54-00165" (at 154.94 48.895 0)
-      (effects (font (size 1.524 1.524)) hide)
-    )
-    (property "Datasheet" "" (at 154.94 55.88 0)
-      (effects (font (size 1.524 1.524)))
-    )
-    (property "Vendor" "Digi-Key" (at 154.94 45.72 0)
-      (effects (font (size 1.524 1.524)) hide)
-    )
-    (property "Vendor Part Number" "839-54-00165CT-ND" (at 154.94 43.18 0)
-      (effects (font (size 1.524 1.524)) hide)
-    )
-    (property "Description" "CONN JACK R/A SMT 5.5X2.5MM" (at 154.94 40.005 0)
-      (effects (font (size 1.524 1.524)) hide)
-    )
-    (property "Manufacturer" "Tensility International Corp" (at 154.94 52.07 0)
-      (effects (font (size 1.27 1.27)) hide)
-    )
-    (property "Manufacturer Part Number" "54-00165" (at 155.575 37.465 0)
-      (effects (font (size 1.27 1.27)) hide)
-    )
-    (property "Sim.Enable" "0" (at 154.94 59.69 0)
-      (effects (font (size 1.27 1.27)) hide)
-    )
-    (pin "1")
-    (pin "2")
-    (pin "3")
-    (instances
-      (project "mouse_joystick_controller"
-        (path "/cc457ebc-4af6-4663-b19f-8cb38f061cb4/f62b8726-10b6-4dce-a8d7-bdccf22557c3"
-          (reference "J2") (unit 1)
-        )
-      )
